Commit message: 备份控制器，还没修弹跳，ird结果

File: rm75_control/rm75_control/control/joint_admittance_8dof/assets/RM75-6F-8dof.slider.generated.urdf (robot description, URDF)
Before this commit: robot RM75-6F-8dof-slider, 14 links, 13 joints
Links:
- link frame_link: geometry visual box size=0.300000 0.998000 0.204000
Joints:
- joint rail_mount: origin xyz=0 0 0.034000 rpy=0 0 0 -> xyz=0 0 0.204000 rpy=0 0 0
