Commit message: RAIL JERK修正。30CM/S

File: rm75_control/rm75_control/assets/robots/rm75_6f_8dof/RM75-6F-8dof.urdf (robot description, URDF)
Before this commit: robot RM75-6F-8dof, 12 links, 11 joints
Joints:
- joint rail_y: limit lower=0.0 upper=0.80 effort=500 velocity=0.20 -> lower=0.0 upper=0.80 effort=500 velocity=0.30
