Commit message: sol2+测试genesis电机联动前备份

File: rm75_control/rm75_control/assets/robots/rm75_6f_8dof/RM75-6F-8dof.genesis.urdf (robot description, URDF)
Before this commit: robot RM75-6F-8dof-genesis, 12 links, 11 joints
Joints:
- joint rail_y: limit lower=-0.18 upper=0.18 effort=500 velocity=0.5 -> lower=0.0 upper=0.80 effort=500 velocity=0.5; origin xyz=0 0 0 rpy=0 0 0 -> xyz=0 -0.4 0 rpy=0 0 0

File: rm75_control/rm75_control/assets/robots/rm75_6f_8dof/RM75-6F-8dof.urdf (robot description, URDF)
Before this commit: robot RM75-6F-8dof, 11 links, 10 joints
Joints:
- joint rail_y: limit lower=-0.25 upper=0.25 effort=500 velocity=0.20 -> lower=0.0 upper=0.80 effort=500 velocity=0.20; origin xyz=0 0 0 rpy=0 0 0 -> xyz=0 -0.4 0 rpy=0 0 0

File: rm75_control/rm75_control/control/joint_admittance_8dof/assets/RM75-6F-8dof.slider.generated.urdf (robot description, URDF)
Before this commit: robot RM75-6F-8dof-slider, 13 links, 12 joints
Links:
- link frame_link: geometry visual box size=0.300000 0.998000 0.200000
- link rail_link: geometry visual box size=0.022000 0.970000 0.018000; visual box size=0.022000 0.970000 0.018000
Joints:
- joint rail_y: limit lower=-0.300000 upper=0.300000 effort=500 velocity=0.20 -> lower=0.000000 upper=0.800000 effort=500 velocity=0.20; origin xyz=0 0 0.066000 rpy=0 0 0 -> xyz=0 -0.400000 0.066000 rpy=0 0 0

Commit message: 标定了除了WRIST之外的

File: rm75_control/rm75_control/assets/robots/rm75_6f_8dof/RM75-6F-8dof.genesis.urdf (robot description, URDF)
Before this commit: robot RM75-6F-8dof-genesis, 13 links, 12 joints
Links:
- added link wrist_camera; visual box size=0.003 0.024 0.003; visual box size=0.004 0.004 0.060
Joints:
- added joint link_7_to_wrist_camera: type fixed, parent link_7, child wrist_camera, origin xyz=0.073036194 0.056181762 0.035658169 rpy=-0.20219080 -0.86145291 1.58824199

File: rm75_control/rm75_control/assets/robots/rm75_6f_8dof/RM75-6F-8dof.urdf (robot description, URDF)
Before this commit: robot RM75-6F-8dof, 12 links, 11 joints
Links:
- added link wrist_camera; visual box size=0.003 0.024 0.003; visual box size=0.004 0.004 0.060
Joints:
- added joint link_7_to_wrist_camera: type fixed, parent link_7, child wrist_camera, origin xyz=0.073036194 0.056181762 0.035658169 rpy=-0.20219080 -0.86145291 1.58824199

File: rm75_control/rm75_control/control/joint_admittance_8dof/assets/RM75-6F-8dof.genesis.urdf (robot description, URDF)
Before this commit: robot RM75-6F-8dof-genesis, 13 links, 12 joints
Links:
- added link wrist_camera; visual box size=0.003 0.024 0.003; visual box size=0.004 0.004 0.060
Joints:
- added joint link_7_to_wrist_camera: type fixed, parent link_7, child wrist_camera, origin xyz=0.073036194 0.056181762 0.035658169 rpy=-0.20219080 -0.86145291 1.58824199

File: rm75_control/rm75_control/control/joint_admittance_8dof/assets/RM75-6F-8dof.slider.generated.urdf (robot description, URDF)
Before this commit: robot RM75-6F-8dof-slider, 14 links, 13 joints
Links:
- added link wrist_camera; visual box size=0.003 0.024 0.003; visual box size=0.004 0.004 0.060
- link frame_link: geometry visual box size=0.500000 0.948000 0.020000
- link rail_link: geometry visual box size=0.016000 0.920000 0.010000; visual box size=0.016000 0.920000 0.010000
- link slider_link: geometry visual box size=0.120000 0.120000 0.226000
Joints:
- added joint link_7_to_wrist_camera: type fixed, parent link_7, child wrist_camera, origin xyz=0.073036194 0.056181762 0.035658169 rpy=-0.20219080 -0.86145291 1.58824199
- joint arm_mount: origin xyz=0.020000 0.000000 0.000000 rpy=0 0 0 -> xyz=0.000000 0.000000 0.000000 rpy=0 0 0
- joint rail_mount: origin xyz=0 0 0.204000 rpy=0 0 0 -> xyz=0 0 0.020000 rpy=0 0 0
- joint rail_y: origin xyz=0 -0.400000 0.066000 rpy=0 0 0 -> xyz=0 -0.400000 0.256000 rpy=0 0 0
