Commit message: 新的横向探头模型加载，备份

File: rm75_control/rm75_control/assets/robots/rm75_6f_8dof/RM75-6F-8dof.collision.urdf (robot description, URDF)
Before this commit: robot RM75-6F-8dof, 11 links, 10 joints
Links:
- added link link_8, mass 0.4829; collision mesh filename=meshes/collision/linear_probe.stl
Joints:
- added joint joint_8: type fixed, parent link_7, child link_8, origin xyz=0 0 0 rpy=0 0 0
- joint link_7_to_tcp: origin xyz=0 0 0.220 rpy=0 0 0 -> xyz=0 -0.08 0.06 rpy=0 1.570796327 -1.570796327

File: rm75_control/rm75_control/assets/robots/rm75_6f_8dof/RM75-6F-8dof.genesis.urdf (robot description, URDF)
Before this commit: robot RM75-6F-8dof-genesis, 12 links, 11 joints
Links:
- added link link_8, mass 0.4829; visual mesh filename=meshes/linear_probe.dae
Joints:
- added joint joint_8: type fixed, parent link_7, child link_8, origin xyz=0 0 0 rpy=0 0 0
- joint link_7_to_tcp: origin xyz=0 0 0.220 rpy=0 0 0 -> xyz=0 -0.08 0.06 rpy=0 1.570796327 -1.570796327

File: rm75_control/rm75_control/assets/robots/rm75_6f_8dof/RM75-6F-8dof.urdf (robot description, URDF)
Before this commit: robot RM75-6F-8dof, 11 links, 10 joints
Links:
- added link link_8, mass 0.4829
Joints:
- added joint joint_8: type fixed, parent link_7, child link_8, origin xyz=0 0 0 rpy=0 0 0
- joint link_7_to_tcp: origin xyz=0 0 0.220 rpy=0 0 0 -> xyz=0 -0.08 0.06 rpy=0 1.570796327 -1.570796327

File: rm75_control/rm75_control/control/joint_admittance_8dof/assets/RM75-6F-8dof.genesis.urdf (robot description, URDF)
Before this commit: robot RM75-6F-8dof-genesis, 12 links, 11 joints
Links:
- added link link_8, mass 0.4829; visual mesh filename=meshes/linear_probe.dae
Joints:
- added joint joint_8: type fixed, parent link_7, child link_8, origin xyz=0 0 0 rpy=0 0 0
- joint link_7_to_tcp: origin xyz=0 0 0.220 rpy=0 0 0 -> xyz=0 -0.08 0.06 rpy=0 1.570796327 -1.570796327

File: rm75_control/rm75_control/control/joint_admittance_8dof/assets/RM75-6F-8dof.slider.generated.urdf (robot description, URDF)
Before this commit: robot RM75-6F-8dof-slider, 13 links, 12 joints
Links:
- added link link_8, mass 0.4829; visual mesh filename=meshes/linear_probe.dae
- link frame_link: geometry visual box size=0.300000 0.998000 0.034000
Joints:
- added joint joint_8: type fixed, parent link_7, child link_8, origin xyz=0 0 0 rpy=0 0 0
- joint link_7_to_tcp: origin xyz=0 0 0.220 rpy=0 0 0 -> xyz=0 -0.08 0.06 rpy=0 1.570796327 -1.570796327
- joint rail_mount: origin xyz=0 0 0.200000 rpy=0 0 0 -> xyz=0 0 0.034000 rpy=0 0 0

Commit message: 修正了探头设计

File: rm75_control/rm75_control/assets/robots/rm75_6f_8dof/RM75-6F-8dof.collision.urdf (robot description, URDF)
Before this commit: robot RM75-6F-8dof, 12 links, 11 joints
Links:
- link link_8: geometry collision mesh filename=meshes/collision/probe45.stl
Joints:
- joint joint_8: origin xyz=0 0 0 rpy=0 0 0 -> xyz=0 0 0 rpy=0 0 3.141592654
- joint link_7_to_tcp: origin xyz=0 -0.08 0.06 rpy=0 1.570796327 -1.570796327 -> xyz=0 -0.01523 0.12135 rpy=0.017732743 0.870791073 -1.547861183

Commit message: bake 时 git e42544f（7/24，commit 信息：V253号称通过…） 体型 20260713_213328（shape_hash=e14c451…） 目录标签 不是 v253_*，是 latest_asset/runs/6/451633f…

File: rm75_control/rm75_control/assets/robots/rm75_6f_8dof/RM75-6F-8dof.collision.urdf (robot description, URDF)
Before this commit: robot RM75-6F-8dof, 12 links, 11 joints
Joints:
- joint rail_y: limit lower=-0.25 upper=0.25 effort=500 velocity=0.20 -> lower=0.0 upper=0.80 effort=500 velocity=0.20; origin xyz=0 0 0 rpy=0 0 0 -> xyz=0 -0.4 0 rpy=0 0 0

Commit message: 关节联动和血管联动确实有进步，比如盆骨的位置终于在骨盆了，有进步。打死你关节还是小问题，脚不全在SMPLX里面，备份控制器准备精简

File: rm75_control/rm75_control/assets/robots/rm75_6f_8dof/RM75-6F-8dof.collision.urdf (robot description, URDF)
Before this commit: robot RM75-6F-8dof, 12 links, 11 joints
Links:
- link link_8: geometry collision mesh filename=meshes/collision/linear_probe.stl
Joints:
- joint joint_8: origin xyz=0 0 0 rpy=0 0 3.141592654 -> xyz=0 0 0 rpy=0 0 0
- joint link_7_to_tcp: origin xyz=0 -0.01523 0.12135 rpy=0.017732743 0.870791073 -1.547861183 -> xyz=0 -0.08 0.06 rpy=0 1.570796327 -1.570796327
- joint rail_y: limit lower=0.0 upper=0.80 effort=500 velocity=0.20 -> lower=-0.25 upper=0.25 effort=500 velocity=0.20; origin xyz=0 -0.4 0 rpy=0 0 0 -> xyz=0 0 0 rpy=0 0 0

File: rm75_control/rm75_control/assets/robots/rm75_6f_8dof/RM75-6F-8dof.genesis.urdf (robot description, URDF)
Before this commit: robot RM75-6F-8dof-genesis, 13 links, 12 joints
Links:
- link link_8: geometry visual mesh filename=meshes/linear_probe.dae
Joints:
- joint joint_8: origin xyz=0 0 0 rpy=0 0 3.141592654 -> xyz=0 0 0 rpy=0 0 0
- joint link_7_to_tcp: origin xyz=0 -0.01523 0.12135 rpy=0.017732743 0.870791073 -1.547861183 -> xyz=0 -0.08 0.06 rpy=0 1.570796327 -1.570796327

File: rm75_control/rm75_control/assets/robots/rm75_6f_8dof/RM75-6F-8dof.urdf (robot description, URDF)
Before this commit: robot RM75-6F-8dof, 12 links, 11 joints
Joints:
- joint joint_8: origin xyz=0 0 0 rpy=0 0 3.141592654 -> xyz=0 0 0 rpy=0 0 0
- joint link_7_to_tcp: origin xyz=0 -0.01523 0.12135 rpy=0.017732743 0.870791073 -1.547861183 -> xyz=0 -0.08 0.06 rpy=0 1.570796327 -1.570796327

File: rm75_control/rm75_control/control/joint_admittance_8dof/assets/RM75-6F-8dof.genesis.urdf (robot description, URDF)
Before this commit: robot RM75-6F-8dof-genesis, 13 links, 12 joints
Links:
- link link_8: geometry visual mesh filename=meshes/linear_probe.dae
Joints:
- joint joint_8: origin xyz=0 0 0 rpy=0 0 3.141592654 -> xyz=0 0 0 rpy=0 0 0
- joint link_7_to_tcp: origin xyz=0 -0.01523 0.12135 rpy=0.017732743 0.870791073 -1.547861183 -> xyz=0 -0.08 0.06 rpy=0 1.570796327 -1.570796327

File: rm75_control/rm75_control/control/joint_admittance_8dof/assets/RM75-6F-8dof.slider.generated.urdf (robot description, URDF)
Before this commit: robot RM75-6F-8dof-slider, 14 links, 13 joints
Links:
- link link_8: geometry visual mesh filename=meshes/linear_probe.dae
Joints:
- joint joint_8: origin xyz=0 0 0 rpy=0 0 3.141592654 -> xyz=0 0 0 rpy=0 0 0
- joint link_7_to_tcp: origin xyz=0 -0.01523 0.12135 rpy=0.017732743 0.870791073 -1.547861183 -> xyz=0 -0.08 0.06 rpy=0 1.570796327 -1.570796327

Commit message: 备份自己的我标定

File: rm75_control/rm75_control/assets/robots/rm75_6f_8dof/RM75-6F-8dof.collision.urdf (robot description, URDF)
Before this commit: robot RM75-6F-8dof, 12 links, 11 joints
Links:
- link link_8: geometry collision mesh filename=meshes/collision/probe45.stl
Joints:
- joint joint_8: origin xyz=0 0 0 rpy=0 0 0 -> xyz=0 0 0 rpy=0 0 3.141592654
- joint link_7_to_tcp: origin xyz=0 -0.08 0.06 rpy=0 1.570796327 -1.570796327 -> xyz=0 -0.01523 0.12135 rpy=0.017732743 0.870791073 -1.547861183

File: rm75_control/rm75_control/assets/robots/rm75_6f_8dof/RM75-6F-8dof.genesis.urdf (robot description, URDF)
Before this commit: robot RM75-6F-8dof-genesis, 13 links, 12 joints
Links:
- link link_8: geometry visual mesh filename=meshes/probe45.dae
Joints:
- joint joint_8: origin xyz=0 0 0 rpy=0 0 0 -> xyz=0 0 0 rpy=0 0 3.141592654
- joint link_7_to_tcp: origin xyz=0 -0.08 0.06 rpy=0 1.570796327 -1.570796327 -> xyz=0 -0.01523 0.12135 rpy=0.017732743 0.870791073 -1.547861183

File: rm75_control/rm75_control/assets/robots/rm75_6f_8dof/RM75-6F-8dof.urdf (robot description, URDF)
Before this commit: robot RM75-6F-8dof, 12 links, 11 joints
Joints:
- joint joint_8: origin xyz=0 0 0 rpy=0 0 0 -> xyz=0 0 0 rpy=0 0 3.141592654
- joint link_7_to_tcp: origin xyz=0 -0.08 0.06 rpy=0 1.570796327 -1.570796327 -> xyz=0 -0.01523 0.12135 rpy=0.017732743 0.870791073 -1.547861183

File: rm75_control/rm75_control/control/joint_admittance_8dof/assets/RM75-6F-8dof.genesis.urdf (robot description, URDF)
Before this commit: robot RM75-6F-8dof-genesis, 13 links, 12 joints
Links:
- link link_8: geometry visual mesh filename=meshes/probe45.dae
Joints:
- joint joint_8: origin xyz=0 0 0 rpy=0 0 0 -> xyz=0 0 0 rpy=0 0 3.141592654
- joint link_7_to_tcp: origin xyz=0 -0.08 0.06 rpy=0 1.570796327 -1.570796327 -> xyz=0 -0.01523 0.12135 rpy=0.017732743 0.870791073 -1.547861183

File: rm75_control/rm75_control/control/joint_admittance_8dof/assets/RM75-6F-8dof.slider.generated.urdf (robot description, URDF)
Before this commit: robot RM75-6F-8dof-slider, 14 links, 13 joints
Links:
- link link_8: geometry visual mesh filename=meshes/probe45.dae
Joints:
- joint joint_8: origin xyz=0 0 0 rpy=0 0 0 -> xyz=0 0 0 rpy=0 0 3.141592654
- joint link_7_to_tcp: origin xyz=0 -0.08 0.06 rpy=0 1.570796327 -1.570796327 -> xyz=0 -0.01523 0.12135 rpy=0.017732743 0.870791073 -1.547861183

Commit message: 标加上激光发布，修光轴标定，联动修了但你不知道怎么样

File: rm75_control/rm75_control/assets/robots/rm75_6f_8dof/RM75-6F-8dof.collision.urdf (robot description, URDF)
Before this commit: robot RM75-6F-8dof, 12 links, 11 joints
Links:
- added link wrist_camera; collision box size=0.12 0.03 0.03
Joints:
- added joint link_7_to_wrist_camera: type fixed, parent link_7, child wrist_camera, origin xyz=0.064853526 0.025247380 0.065670289 rpy=-0.19092023 -0.86158535 1.58594946

File: rm75_control/rm75_control/assets/robots/rm75_6f_8dof/RM75-6F-8dof.genesis.urdf (robot description, URDF)
Before this commit: robot RM75-6F-8dof-genesis, 14 links, 13 joints
Links:
- removed link wrist_camera
Joints:
- removed joint link_7_to_wrist_camera

File: rm75_control/rm75_control/assets/robots/rm75_6f_8dof/RM75-6F-8dof.urdf (robot description, URDF)
Before this commit: robot RM75-6F-8dof, 13 links, 12 joints
Links:
- link wrist_camera: geometry 
Joints:
- joint link_7_to_wrist_camera: origin xyz=0.073036194 0.056181762 0.035658169 rpy=-0.20219080 -0.86145291 1.58824199 -> xyz=0.064853526 0.025247380 0.065670289 rpy=-0.19092023 -0.86158535 1.58594946

File: rm75_control/rm75_control/control/joint_admittance_8dof/assets/RM75-6F-8dof.genesis.urdf (robot description, URDF)
Before this commit: robot RM75-6F-8dof-genesis, 14 links, 13 joints
Links:
- removed link wrist_camera
Joints:
- removed joint link_7_to_wrist_camera

File: rm75_control/rm75_control/control/joint_admittance_8dof/assets/RM75-6F-8dof.slider.generated.urdf (robot description, URDF)
Before this commit: robot RM75-6F-8dof-slider, 15 links, 14 joints
Links:
- link wrist_camera: geometry collision box size=0.12 0.03 0.03
Joints:
- joint link_7_to_wrist_camera: origin xyz=0.073036194 0.056181762 0.035658169 rpy=-0.20219080 -0.86145291 1.58824199 -> xyz=0.064853526 0.025247380 0.065670289 rpy=-0.19092023 -0.86158535 1.58594946
